File: cpu6502/pcb6502/pcb6502.kicad_pcb (KiCad board)
At the start: 2 copper layers, 111.8 x 109.2 mm, 34 parts, among them J1 Power, J2 RS232, J3 VIA PA, J4 VIA PB, J5 Ext RST, SW1 Reset, U1 6502, U2 EEPROM, U3 RAM, U4 65C22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

Commit message: Finished the PCB
Parts:
- removed Y1: Crystal, Crystal:Crystal_HC49-4H_Vertical
- added 1.8432 mhz: Crystal, Crystal:Crystal_HC49-4H_Vertical, F.Cu at (157.7, 132.1)
- C6: value 20pf -> 20pf
- U7: value W65C51NxP -> W65C51N
- moved H3 164.7 mm to (55.9, 134.8)
- moved H1 101.6 mm to (144.6, 50.8)
- moved R4 100.1 mm to (148.6, 132.1)
- moved U6 82.6 mm to (179.2, 68.6), turned to -90 degrees
- moved J5 80.7 mm to (96.5, 58.4), turned to -90 degrees
- moved U8 77.3 mm to (165.6, 124.5), turned to 180 degrees
- moved J1 76.3 mm to (169.3, 56.8), turned to 180 degrees
- moved C2 75.5 mm to (175.3, 124.5), turned to 180 degrees
- moved D2 71.3 mm to (134.6, 132.1), turned to 180 degrees
- moved C3 68.4 mm to (175.2, 119.4), turned to 180 degrees
- moved D3 63.7 mm to (160.0, 55.9)
- moved C8 63.5 mm to (177.8, 63.5)
- moved C6 61.0 mm to (172.7, 114.3)
- moved C4 60.6 mm to (175.3, 104.1), turned to 180 degrees
- moved U7 57.7 mm to (149.4, 107.1)
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Routing:
- net GND: track 627.5 -> 0.00 mm, vias 6 -> 0
- net +5V: track 397.7 -> 2.54 mm, vias 2 -> 0
- net Net-(J5-Pin_1): track 168.8 -> 28.2 mm
- net /RST: track 187.3 -> 280.4 mm, vias 3 -> 1
- net /IRQ: track 92.9 -> 153.4 mm
- net /A12: track 96.9 -> 148.7 mm
- net /A10: track 56.0 -> 104.2 mm, vias 1 -> 0
- net /A11: track 67.9 -> 114.1 mm
- net /XTAL2: track 30.7 -> 76.1 mm
- net /A9: track 66.9 -> 111.7 mm
- net /A13: track 95.3 -> 136.3 mm, vias 2 -> 1
- net /A8: track 74.1 -> 111.6 mm
- net /A0: track 178.6 -> 141.2 mm, vias 1 -> 0
- net /PHI2: track 220.5 -> 256.0 mm, vias 1 -> 2
- net /PA1: track 13.3 -> 47.2 mm
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- added copper zone on In2.Cu, net +5V
- added copper zone on In1.Cu, net GND
- removed copper zone on B.Cu, net GND
- removed copper zone on F.Cu, net GND
Other:
- board size 111.8 x 109.2 mm -> 134.6 x 94 mm
- copper layers 2 -> 4
- board text added: "+5V"
- board text added: "-"
- board text added: "0"
- board text added: "1"
- board text added: "2"
- board text added: "3"
- board text added: "4"
- board text added: "5"
- board text added: "5-12v Input"
- board text added: "6"
- board text added: "6502 CPU, RS232, VIA"
- board text added: "7"
- board text added: "C1"
- board text added: "C2"
- board text added: "Chris Gall, 2023, v1.0"
- board text removed: "5V"
- board text removed: "CA1"
- board text removed: "CA2"
- board text removed: "CB1"
- board text removed: "CB2"
- board text removed: "CG 6502 / RS232 Revision 1.0 2023"
- board text removed: "GND"
- board text removed: "PA0"
- board text removed: "PA1"
- board text removed: "PA2"
- board text removed: "PA3"
- board text removed: "PA4"
- board text removed: "PA5"
- board text removed: "PA6"
- board text removed: "PA7"
- board text removed: "PB0"
- board text removed: "PB1"
- board text removed: "PB2"
- board text removed: "PB3"
- board text removed: "PB4"
- board text removed: "PB5"
- board text removed: "PB6"
- board text removed: "PB7"

Commit message: Finalizing pcb
Parts:
- added J6: Address, Connector_PinHeader_2.54mm:PinHeader_2x08_P2.54mm_Vertical, F.Cu at (119.4, 53.3)
- added J7: Data, Connector_PinHeader_2.54mm:PinHeader_2x04_P2.54mm_Vertical, F.Cu at (101.6, 53.3)
- added J8: CPU, Connector_PinHeader_2.54mm:PinHeader_2x04_P2.54mm_Vertical, F.Cu at (83.8, 53.3)
- added J9: Interrupt Enable, Connector_PinHeader_2.54mm:PinHeader_2x06_P2.54mm_Vertical, F.Cu at (66.0, 53.3)
- C6: value 20pf -> 20pf
- U1: value 6502 -> 6502 (CPU)
- U2: value EEPROM -> 28C256 (EEPROM)
- U3: value RAM -> 62256 (RAM)
- U4: value 65C22 -> 6522 (VIA)
- U7: value W65C51N -> 6551 (UART)
- U9: value ~ -> DS1813
- Y1: renamed from 1.8432 mhz
- moved R2 69.9 mm to (123.2, 132.1), turned to 0 degrees
- moved D1 66.6 mm to (115.6, 132.1)
- moved H1 35.9 mm to (180.5, 48.3)
- moved D2 10.2 mm to (144.8, 132.1)
- moved R4 8.89 mm to (157.5, 132.1)
- moved Y1 7.42 mm to (165.1, 132.1)
- moved J5 5.68 mm to (99.1, 63.5)
- moved SW1 3.80 mm to (84.9, 61.5)
- moved D3 2.54 mm to (160.0, 53.3)
- moved U9 2.54 mm to (83.8, 73.7)
Connections:
- D2 pad 2: /IRQ -> /ACIAIRQ
- U1 pad 6: +5V -> /NMI
- U4 pad 21: /IRQ -> /VIAIRQ
Routing:
- net /ACIAIRQ: track 0.00 -> 155.3 mm, vias 0 -> 1
- net /IRQ: track 153.4 -> 55.8 mm, vias 1 -> 0
- net /R/W: track 186.2 -> 276.1 mm
- net /VIAIRQ: track 0.00 -> 81.2 mm, vias 0 -> 1
- net /D7: track 152.8 -> 216.2 mm
- net /D6: track 147.4 -> 203.8 mm
- net /A10: track 104.2 -> 160.5 mm
- net /A13: track 136.3 -> 187.7 mm
- net /D5: track 141.9 -> 191.4 mm
- net /D3: track 131.0 -> 174.2 mm
- net /D4: track 136.4 -> 178.4 mm
- net /A14: track 144.0 -> 182.4 mm
- net /NMI: track 0.00 -> 38.3 mm
- net /PHI2: track 256.0 -> 293.2 mm
- net /A12: track 148.7 -> 178.4 mm
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Other:
- board size 134.6 x 94 mm -> 134.6 x 96.5 mm
- board text added: "5-12v Input (center +)"
- board text added: "6502 with VIA and RS232 Chris Gall, 2023, v1.0"
- board text added: "A0"
- board text added: "A1"
- board text added: "A10"
- board text added: "A11"
- board text added: "A12"
- board text added: "A13"
- board text added: "A14"
- board text added: "A2"
- board text added: "A3"
- board text added: "A4"
- board text added: "A5"
- board text added: "A6"
- board text added: "A7"
- board text added: "A8"
- board text added: "A9"
- board text added: "ACIA"
- board text added: "D0"
- board text added: "D1"
- board text added: "D2"
- board text added: "D3"
- board text added: "D4"
- board text added: "D5"
- board text added: "D6"
- board text added: "D7"
- board text added: "Ext IRQ"
- board text added: "Ext NMI"
- board text added: "IRQ"
- board text added: "Jmp Required for IRQ and NMI"
- board text added: "NC"
- board text added: "NMI"
- board text added: "No IRQ"
- board text added: "No NMI"
- board text added: "PHI"
- board text added: "R/W"
- board text added: "RST"
- board text added: "VIA"
- board text removed: "5-12v Input"
- board text removed: "6502 CPU, RS232, VIA"
- board text removed: "Chris Gall, 2023, v1.0"

Commit message: Cleanup routes
Routing:
- net /RST: track 288.3 -> 263.2 mm, vias 1 -> 2
- net /A12: track 178.4 -> 172.7 mm
- net /CS2: track 136.7 -> 140.7 mm
- net /PHI2: track 293.2 -> 296.8 mm
- net /CS_RAM: track 49.3 -> 52.2 mm, vias 0 -> 1
- net /A0: track 156.6 -> 159.0 mm
- net /A4: track 112.7 -> 114.0 mm
- net /A1: track 167.6 -> 169.0 mm
- net /A2: track 149.6 -> 150.9 mm
- net /A6: track 122.8 -> 124.2 mm
- net /A5: track 117.4 -> 118.7 mm
- net /A7: track 128.3 -> 129.6 mm
- net /A3: track 155.8 -> 157.1 mm
